File: STM32F4Example/STM32F4Example.kicad_sch (KiCad schematic)
At the start: 23 parts, among them J1 Conn_01x02_Pin, J2 Conn_01x17_Pin, J3 Conn_01x17_Pin, P1 USB_C_Plug_USB2.0, U1 STM32F411CCUx, U2 AZ1117H-3.3TRG1, X1 X322512MSB4SI

Commit message: traces
Parts:
- removed C10: 100nF, symbol Device:C
- removed P1: USB_C_Plug_USB2.0, symbol Connector:USB_C_Plug_USB2.0
- removed U1: STM32F411CCUx, Package_CSP:ST_WLCSP-36_Die458, symbol MCU_ST_STM32F4:STM32F411CCUx
- added R3: 5K1, Resistor_SMD:R_0603_1608Metric, symbol Device:R
- added U3: GT-USB-7010ASV, gt-usb-7010:USB-C-SMD_G-SWITCH_GT-USB-7010ASV, symbol gt-usb-7010:GT-USB-7010ASV
- added U4: STM32F411CCUx, Package_DFN_QFN:QFN-48-1EP_7x7mm_P0.5mm_EP5.6x5.6mm, symbol MCU_ST_STM32F4:STM32F411CCUx
- C1, C11, C12, C13, C2, C3, C4, C5, C6, C7, C8, C9: footprint (none) -> Capacitor_SMD:C_0402_1005Metric
- J2, J3: footprint Connector_PinSocket_2.54mm:PinSocket_1x17_P2.54mm_Vertical -> Connector_PinHeader_2.54mm:PinHeader_1x17_P2.54mm_Vertical
- L1: footprint (none) -> Inductor_SMD:L_0603_1608Metric
- R1, R2: footprint (none) -> Resistor_SMD:R_0603_1608Metric
Connections:
- net +3.3VA: now also U4.9 (VDDA)
- net +3V3: now also U4.1 (VBAT), U4.24 (VDD), U4.36 (VDD), U4.48 (VDD)
- net +5V: now also U3.A4B9 (VBUS), U3.B4A9 (VBUS)
- net GND: now also R3.2, U3.A1B12 (GND), U3.B1A12 (GND), U4.23 (VSS), U4.35 (VSS), U4.47 (VSS), U4.49 (VSS), U4.8 (VSSA)
- net USBD+: now also U3.A6 (DP1), U3.B6 (DP2), U4.33 (PA12)
- net USBD-: now also U3.A7 (DN1), U3.B7 (DN2), U4.32 (PA11)
- net XIN: now also U4.5 (PH0)
- net XOT: now also U4.6 (PH1)
- net at R1.1: now also U3.B5 (CC2)
- net at J1.2 (Pin_2), R2.1: now also U4.44 (BOOT0)
- net at J2.10 (Pin_10): now also U4.45 (PB8)
- net at J2.11 (Pin_11): now also U4.46 (PB9)
- net at J2.12 (Pin_12): now also U4.21 (PB10)
- net at J2.13 (Pin_13): now also U4.25 (PB12)
- net at J2.14 (Pin_14): now also U4.26 (PB13)
- net at J2.15 (Pin_15): now also U4.27 (PB14)
- net at J2.16 (Pin_16): now also U4.28 (PB15)
- net at J2.2 (Pin_2): now also U4.18 (PB0)
- net at J2.3 (Pin_3): now also U4.19 (PB1)
- net at J2.4 (Pin_4): now also U4.20 (PB2)
- net at J2.5 (Pin_5): now also U4.39 (PB3)
- net at J2.6 (Pin_6): now also U4.40 (PB4)
- net at J2.7 (Pin_7): now also U4.41 (PB5)
- net at J2.8 (Pin_8): now also U4.42 (PB6)
- net at J2.9 (Pin_9): now also U4.43 (PB7)
- net at C13.1: now also U4.22 (VCAP1)
- net at C1.1: now also U4.7 (NRST)
- net at J3.10 (Pin_10): now also U4.17 (PA7)
- net at J3.11 (Pin_11): now also U4.16 (PA6)
- net at J3.12 (Pin_12): now also U4.15 (PA5)
- net at J3.13 (Pin_13): now also U4.14 (PA4)
- net at J3.14 (Pin_14): now also U4.13 (PA3)
- net at J3.15 (Pin_15): now also U4.12 (PA2)
- net at J3.16 (Pin_16): now also U4.11 (PA1)
- net at J3.2 (Pin_2): now also U4.38 (PA15)
- net at J3.3 (Pin_3): now also U4.37 (PA14)
- net at J3.4 (Pin_4): now also U4.34 (PA13)
- net at J3.7 (Pin_7): now also U4.31 (PA10)
- net at J3.8 (Pin_8): now also U4.30 (PA9)
- net at J3.9 (Pin_9): now also U4.29 (PA8)
- new net: R3.1, U3.A5 (CC1)
- no-connect marks 6 -> 10
Other:
- note added: "USB C connector for power delivery & prog"
- note removed: "USB C plug for power and prog"
