File: STM32F4Example/STM32F4Example.kicad_pcb (KiCad board)
At the start: 2 copper layers, 27 x 44.7 mm, 23 parts, among them J1 Conn_01x02_Pin, J2 Conn_01x17_Pin, J3 Conn_01x17_Pin, U2 AZ1117H-3.3TRG1, U3 GT-USB-7010ASV, U4 STM32F411CCUx, X1 X322512MSB4SI

Commit message: new switch & board in production
Parts:
- added C10: 10uF, Capacitor_SMD:C_0402_1005Metric, F.Cu at (107.5, 99.4)
- C12: value 20uF -> 10uF
- L1: value 3nH -> 10uH
- moved C12 0.10 mm to (107.5, 100.4)
Routing:
- net /USBD+: track 27.1 -> 28.5 mm
- net +3V3: track 152.8 -> 154.1 mm
